File: KiCad/Midea WiFi Dongle.kicad_sch (KiCad schematic)
At the start: 16 parts, among them J1 USB_A, Q1 BSS138, Q2 BSS138, SW1 SW_Push, SW2 SW_Push, U1 AMS1117-3.3, U2 ESP-12F

Commit message: Added files for v2r1; updated ReadMe
Parts:
- removed C2: 470pF, Capacitor_SMD:C_0402_1005Metric_Pad0.74x0.62mm_HandSolder, symbol Device:C
- renumbered C3 to C2, C4 to C3
Changed lines of the file:
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@@
 	(wire
 		(pts
-			(xy 116.84 153.67) (xy 116.84 158.75)
+			(xy 63.5 91.44) (xy 73.66 91.44)
 		)
 		(stroke
@@
 	(wire
 		(pts
-			(xy 116.84 166.37) (xy 116.84 167.64)
+			(xy 125.73 133.35) (xy 134.62 133.35)
 		)
 		(stroke
@@
 	(wire
 		(pts
-			(xy 63.5 91.44) (xy 73.66 91.44)
-		)
-		(stroke
-			(width 0)
-			(type default)
-		)
-	)
-	(wire
-		(pts
-			(xy 125.73 133.35) (xy 134.62 133.35)
-		)
-		(stroke
-			(width 0)
-			(type default)
-		)
-	)
-	(wire
-		(pts
 			(xy 73.66 91.44) (xy 83.82 91.44)
-		)
-		(stroke
-			(width 0)
-			(type default)
-		)
-	)
-	(wire
-		(pts
-			(xy 105.41 153.67) (xy 116.84 153.67)
 		)
 		(stroke
@@
 	)
 	(label "RESET"
-		(at 111.76 153.67 180)
+		(at 105.41 153.67 0)
 		(effects
 			(font
 				(size 1.27 1.27)
 			)
-			(justify right bottom)
+			(justify left bottom)
 		)
 	)
@@
 		(on_board yes)
 		(dnp no)
-		(property "Reference" "C4"
+		(property "Reference" "C3"
 			(at 154.94 54.5592 90)
 			(effects
@@
 			(project "Midea WiFi Dongle"
 				(path "/ee1d3c30-6791-41bb-a985-8c603430de03"
-					(reference "C4")
+					(reference "C3")
 					(unit 1)
 				)
@@
 		(on_board yes)
 		(dnp no)
-		(property "Reference" "C3"
+		(property "Reference" "C2"
 			(at 86.8172 86.4616 0)
 			(effects
@@
 			(project "Midea WiFi Dongle"
 				(path "/ee1d3c30-6791-41bb-a985-8c603430de03"
-					(reference "C3")
+					(reference "C2")
 					(unit 1)
 				)
@@
 			)
 		)
-		(property "Description" ""
+		(property "Description" "3x4mm"
 			(at 207.01 111.76 0)
 			(effects
@@
 				(path "/ee1d3c30-6791-41bb-a985-8c603430de03"
 					(reference "#PWR03")
-					(unit 1)
-				)
-			)
-		)
-	)
-	(symbol
-		(lib_id "Device:C")
-		(at 116.84 162.56 0)
-		(unit 1)
-		(exclude_from_sim no)
-		(in_bom yes)
-		(on_board yes)
-		(dnp no)
-		(property "Reference" "C2"
-			(at 119.761 161.3916 0)
-			(effects
-				(font
-					(size 1.27 1.27)
-				)
-				(justify left)
-			)
-		)
-		(property "Value" "470pF"
-			(at 119.761 163.703 0)
-			(effects
-				(font
-					(size 1.27 1.27)
-				)
-				(justify left)
-			)
-		)
-		(property "Footprint" "Capacitor_SMD:C_0402_1005Metric_Pad0.74x0.62mm_HandSolder"
-			(at 117.8052 166.37 0)
-			(effects
-				(font
-					(size 1.27 1.27)
-				)
-				(hide yes)
-			)
-		)
-		(property "Datasheet" "~"
-			(at 116.84 162.56 0)
-			(effects
-				(font
-					(size 1.27 1.27)
-				)
-				(hide yes)
-			)
-		)
-		(property "Description" ""
-			(at 116.84 162.56 0)
-			(effects
-				(font
-					(size 1.27 1.27)
-				)
-				(hide yes)
-			)
-		)
-		(pin "1"
-		)
-		(pin "2"
-		)
-		(instances
-			(project "Midea WiFi Dongle"
-				(path "/ee1d3c30-6791-41bb-a985-8c603430de03"
-					(reference "C2")
 					(unit 1)
 				)
@@
 			)
 		)
-		(property "Description" ""
+		(property "Description" "3x4mm"
 			(at 207.01 125.73 0)
 			(effects
@@
 					(unit 1)
 				)
-			)
-		)
-	)
-	(symbol
-		(lib_id "power:GND")
-		(at 116.84 167.64 0)
-		(unit 1)
-		(exclude_from_sim no)
-		(in_bom yes)
-		(on_board yes)
-		(dnp no)
-		(property "Reference" "#PWR02"
-			(at 116.84 173.99 0)
-			(effects
-				(font
-					(size 1.27 1.27)
-				)
-				(hide yes)
-			)
-		)
-		(property "Value" "GND"
-			(at 116.967 172.0342 0)
-			(effects
-				(font
-					(size 1.27 1.27)
-				)
-			)
-		)
-		(property "Footprint" ""
-			(at 116.84 167.64 0)
-			(effects
-				(font
-					(size 1.27 1.27)
-				)
-				(hide yes)
-			)
-		)
-		(property "Datasheet" ""
-			(at 116.84 167.64 0)
-			(effects
-				(font
-					(size 1.27 1.27)
-				)
-				(hide yes)
-			)
-		)
-		(property "Description" ""
-			(at 116.84 167.64 0)
-			(effects
-				(font
-					(size 1.27 1.27)
-				)
-				(hide yes)
-			)
-		)
-		(pin "1"
-		)
-		(instances
-			(project "Midea WiFi Dongle"
-				(path "/ee1d3c30-6791-41bb-a985-8c603430de03"
-					(reference "#PWR02")
-					(unit 1)
-				)

Commit message: Updated iBOM
Parts:
- RN1: value R_Pack04 -> 10k
Changed lines of the file:
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@@
 			)
 		)
-		(property "Description" ""
+		(property "Description" "Can be ceramic or tantalum, 2012 metric equals 0805 imperial"
 			(at 83.82 87.63 0)
 			(effects
@@
 			)
 		)
-		(property "Description" ""
+		(property "Description" "Can be ceramic or tantalum, 2012 metric equals 0805 imperial"
 			(at 63.5 87.63 0)
 			(effects
@@
 			)
 		)
-		(property "Value" "R_Pack04"
+		(property "Value" "10k"
 			(at 98.425 163.83 0)
 			(effects
